Commit message: web2_update_radiation_nav_optimization_baseline_rad

File: smart_master/urdf/full_system.urdf.xacro (robot description, xacro)
@@ -15,5 +15,5 @@
       <!-- Attention. "arm_base_link" is the actual name of the root link of arm from manipulator.urdf.xacro -->
       <child link="arm_base_link"/>
-      <origin xyz="0.1 -0.03 -0.02" rpy="0 0 1.5708"/>
+      <origin xyz="0.1 -0.03 -0.02" rpy="0 0 0"/>
     </joint>
   </xacro:if>

File: smart_sim2real/urdf/sim_wrapper.urdf.xacro (robot description, xacro)
@@ -9,5 +9,4 @@
     <xacro:include filename="$(find ugv_tracked_description)/urdf/sensors/plugins.urdf.xacro" />
     <xacro:include filename="$(find ugv_tracked_description)/urdf/controllers/diff_drive.urdf.xacro" />
-    <!-- Gazebo plugin only for simulation assembly -->
     <xacro:if value="$(arg use_arm)">
         <gazebo>
@@ -15,5 +14,4 @@
                 <!-- load controllers from the new common config -->
                 <parameters>$(find smart_moveit_config)/config/ros2_controllers.yaml</parameters>
-                <!-- Redirect topic for the smart mixer (so the arm doesn't shake and wheels are present) -->
                 <ros>
                     <remapping>/joint_states:=/arm_joint_states</remapping>
